File: overall/Smart Glove Breakout/overall_connections.brd (EAGLE design)
At the start: 100.3 x 64.8 mm, 15 parts, among them IC1 LD1085

Commit message: Revised PCB design
Fixed error with voltage regulator pinout, package pins for our device
did not match the Eagle schematic. Also routed V+ pins to both the mbed
device and the Huzzah IC.
Parts:
- C1, C2: device rcl:C1206 -> rcl:E1,8-4
- IC1: device linear:TO220H -> smart_glove_breakout:TO220H
- moved IC1 2.54 mm to (40.6, 11.4)
- moved C1 2.03 mm to (57.1, 8.13)
- moved C2 1.80 mm to (63.5, 3.81)
- moved G1 1.27 mm to (63.5, 12.7)
Connections:
- removed net VIN: KIT1.VIN
- net +5V: now also C2.+, IC1.2, KIT1.VIN, U$2.P$8; no longer C2.1, IC1.3
- net GND: now also C1.-, C2.-, IC1.3; no longer C1.2, C2.2, IC1.2
- net N$10: now also C1.+; no longer C1.1
Routing:
- net GND: track 114.6 -> 20.3 mm
- net +5V: track 57.2 -> 115.6 mm
- net VCC: track 142.5 -> 130.2 mm
- net N$10: track 17.1 -> 18.2 mm
